File: ServerPSU_Breakout.sch (KiCad schematic (older format))
At the start: 2 parts

Commit message: updated schematic
Switched single point outputs to 6 pin outputs
Parts:
- removed J?: Conn_01x02, symbol Connector_Generic:Conn_01x02
- added J_DATA1: Conn_02x06_Counter_Clockwise, symbol Connector_Generic:Conn_02x06_Counter_Clockwise
- added J_GND1, J_VOUT1: 5.08mm, symbol Connector_Generic:Conn_01x06
Connections:
- wire segments 119 -> 156
Other:
- moved on the sheet: J_PSU_IN1

Commit message: Created Layout
Parts:
- removed J_DATA1: Conn_02x06_Counter_Clockwise, symbol Connector_Generic:Conn_02x06_Counter_Clockwise
- added J_DATA1: 1x10_2.54mm, Connector_PinHeader_2.54mm:PinHeader_1x10_P2.54mm_Horizontal, symbol Connector_Generic:Conn_01x10
- J_GND1, J_VOUT1: value 5.08mm -> 1x6_5.08mm; footprint (none) -> Samtec HPM-06-02-T-S-RA_1x6:Samtec HPM-06-02-T-S-RA_2x6
- J_PSU_IN1: value Conn_02x32_Counter_Clockwise -> Amphenol FCI 10046971-001LF; footprint (none) -> Amphenol FCI 10046971-001LF_2x32:Amphenol_FCI_10046971-001LF_2x32
Changed lines of the file:
@@
 P 2100 3100
 F 0 "J_PSU_IN1" H 2100 4800 50  0000 C CNN
-F 1 "Conn_02x32_Counter_Clockwise" H 2150 4725 50  0001 C CNN
-F 2 "" H 2100 3100 50  0001 C CNN
+F 1 "Amphenol FCI 10046971-001LF" H 2150 4725 50  0001 C CNN
+F 2 "Amphenol FCI 10046971-001LF_2x32:Amphenol_FCI_10046971-001LF_2x32" H 2100 3100 50  0001 C CNN
 F 3 "~" H 2100 3100 50  0001 C CNN
 	1    2100 3100
@@
 Text Label 3200 4200 2    50   ~ 0
 PSINTERRUPT
-$Comp
-L Connector_Generic:Conn_02x06_Counter_Clockwise J_DATA1
-U 1 1 5C6EAFA4
-P 6100 4400
-F 0 "J_DATA1" H 6150 4725 50  0000 C CNN
-F 1 "Conn_02x06_Counter_Clockwise" H 6150 4726 50  0001 C CNN
-F 2 "" H 6100 4400 50  0001 C CNN
-F 3 "~" H 6100 4400 50  0001 C CNN
-	1    6100 4400
-	1    0    0    -1
-$EndComp
 Wire Wire Line
 	5650 2000 5350 2000
@@
 GND
 Wire Wire Line
-	7200 4200 6400 4200
-Wire Wire Line
-	7200 4300 6400 4300
-Wire Wire Line
-	7200 4400 6400 4400
-Wire Wire Line
-	7200 4500 6400 4500
-Wire Wire Line
-	7200 4600 6400 4600
-Wire Wire Line
-	6400 4700 7200 4700
-Text Label 7200 4700 2    50   ~ 0
+	5450 4200 5950 4200
+Wire Wire Line
+	5450 4300 5950 4300
+Wire Wire Line
+	5450 4400 5950 4400
+Wire Wire Line
+	5450 4500 5950 4500
+Wire Wire Line
+	5450 4600 5950 4600
+Wire Wire Line
+	5950 4700 5450 4700
+Text Label 5450 4700 0    50   ~ 0
 PSON
-Text Label 7200 4600 2    50   ~ 0
+Text Label 5450 4600 0    50   ~ 0
 ISHARE
-Text Label 7200 4500 2    50   ~ 0
+Text Label 5450 4500 0    50   ~ 0
 PSOK
-Text Label 7200 4400 2    50   ~ 0
+Text Label 5450 4400 0    50   ~ 0
 PRESENT
-Text Label 7200 4300 2    50   ~ 0
+Text Label 5450 4300 0    50   ~ 0
 12VSB
-Text Label 7200 4200 2    50   ~ 0
+Text Label 5450 4200 0    50   ~ 0
 PSINTERRUPT
 Wire Wire Line
-	5900 4200 5400 4200
-Wire Wire Line
-	5900 4600 5400 4600
-Wire Wire Line
-	5900 4700 5400 4700
-Text Label 5400 4200 0    50   ~ 0
+	5950 3800 5450 3800
+Wire Wire Line
+	5950 4000 5450 4000
+Wire Wire Line
+	5950 4100 5450 4100
+Text Label 5450 3800 0    50   ~ 0
 ADDR
 Wire Wire Line
-	5900 4500 5200 4500
-Wire Wire Line
-	5200 4900 5200 4500
-Text Label 5200 4900 1    50   ~ 0
+	5950 3900 5250 3900
+Wire Wire Line
+	5250 4300 5250 3900
+Text Label 5250 4300 1    50   ~ 0
 GND
-Text Label 5400 4700 0    50   ~ 0
+Text Label 5450 4100 0    50   ~ 0
 SDA
-Text Label 5400 4600 0    50   ~ 0
+Text Label 5450 4000 0    50   ~ 0
 SCL
 $Comp
@@
 P 6150 2000
 F 0 "J_VOUT1" H 6229 1992 50  0000 L CNN
-F 1 "5.08mm" H 6229 1901 50  0000 L CNN
-F 2 "" H 6150 2000 50  0001 C CNN
+F 1 "1x6_5.08mm" H 6229 1901 50  0000 L CNN
+F 2 "Samtec HPM-06-02-T-S-RA_1x6:Samtec HPM-06-02-T-S-RA_2x6" H 6150 2000 50  0001 C CNN
 F 3 "~" H 6150 2000 50  0001 C CNN
 	1    6150 2000
@@
 P 6150 2900
 F 0 "J_GND1" H 6229 2892 50  0000 L CNN
-F 1 "5.08mm" H 6229 2801 50  0000 L CNN
-F 2 "" H 6150 2900 50  0001 C CNN
+F 1 "1x6_5.08mm" H 6229 2801 50  0000 L CNN
+F 2 "Samtec HPM-06-02-T-S-RA_1x6:Samtec HPM-06-02-T-S-RA_2x6" H 6150 2900 50  0001 C CNN
 F 3 "~" H 6150 2900 50  0001 C CNN
 	1    6150 2900
@@
 Wire Wire Line
 	5250 2900 5650 2900
+$Comp
+L Connector_Generic:Conn_01x10 J_DATA1
+U 1 1 5C7060C6
+P 6150 4200
+F 0 "J_DATA1" H 6230 4192 50  0000 L CNN
+F 1 "1x10_2.54mm" H 6230 4101 50  0000 L CNN
+F 2 "Connector_PinHeader_2.54mm:PinHeader_1x10_P2.54mm_Horizontal" H 6150 4200 50  0001 C CNN
+F 3 "~" H 6150 4200 50  0001 C CNN
+	1    6150 4200
+	1    0    0    -1
+$EndComp
 $EndSCHEMATC

Commit message: update
Parts:
- removed J_DATA1: 1x10_2.54mm, Connector_PinHeader_2.54mm:PinHeader_1x10_P2.54mm_Horizontal, symbol Connector_Generic:Conn_01x10
- added J_DATA1: 2x5_2.54mm, Connector_PinHeader_2.54mm:PinHeader_2x05_P2.54mm_Vertical, symbol Connector_Generic:Conn_02x05_Odd_Even
Changed lines of the file:
@@
 GND
 Wire Wire Line
-	5450 4200 5950 4200
+	6900 4550 6400 4550
 Wire Wire Line
-	5450 4300 5950 4300
+	6900 4450 6400 4450
 Wire Wire Line
-	5450 4400 5950 4400
+	6900 4350 6400 4350
 Wire Wire Line
-	5450 4500 5950 4500
+	6900 4250 6400 4250
 Wire Wire Line
-	5450 4600 5950 4600
+	6900 4150 6400 4150
 Wire Wire Line
-	5950 4700 5450 4700
-Text Label 5450 4700 0    50   ~ 0
+	5900 4150 5400 4150
+Text Label 5400 4150 0    50   ~ 0
 PSON
-Text Label 5450 4600 0    50   ~ 0
+Text Label 6900 4150 2    50   ~ 0
 ISHARE
-Text Label 5450 4500 0    50   ~ 0
+Text Label 6900 4250 2    50   ~ 0
 PSOK
-Text Label 5450 4400 0    50   ~ 0
+Text Label 6900 4350 2    50   ~ 0
 PRESENT
-Text Label 5450 4300 0    50   ~ 0
+Text Label 6900 4450 2    50   ~ 0
 12VSB
-Text Label 5450 4200 0    50   ~ 0
+Text Label 6900 4550 2    50   ~ 0
 PSINTERRUPT
 Wire Wire Line
-	5950 3800 5450 3800
+	5900 4450 5400 4450
 Wire Wire Line
-	5950 4000 5450 4000
+	5900 4350 5400 4350
 Wire Wire Line
-	5950 4100 5450 4100
-Text Label 5450 3800 0    50   ~ 0
+	5900 4250 5400 4250
+Text Label 5400 4450 0    50   ~ 0
 ADDR
 Wire Wire Line
-	5950 3900 5250 3900
+	5900 4550 5200 4550
 Wire Wire Line
-	5250 4300 5250 3900
-Text Label 5250 4300 1    50   ~ 0
+	5200 4850 5200 4550
+Text Label 5200 4850 1    50   ~ 0
 GND
-Text Label 5450 4100 0    50   ~ 0
+Text Label 5400 4250 0    50   ~ 0
 SDA
-Text Label 5450 4000 0    50   ~ 0
+Text Label 5400 4350 0    50   ~ 0
 SCL
 $Comp
@@
 	5250 2900 5650 2900
 $Comp
-L Connector_Generic:Conn_01x10 J_DATA1
-U 1 1 5C7060C6
-P 6150 4200
-F 0 "J_DATA1" H 6230 4192 50  0000 L CNN
-F 1 "1x10_2.54mm" H 6230 4101 50  0000 L CNN
-F 2 "Connector_PinHeader_2.54mm:PinHeader_1x10_P2.54mm_Horizontal" H 6150 4200 50  0001 C CNN
-F 3 "~" H 6150 4200 50  0001 C CNN
-	1    6150 4200
+L Connector_Generic:Conn_02x05_Odd_Even J_DATA1
+U 1 1 5C74C643
+P 6100 4350
+F 0 "J_DATA1" H 6150 4767 50  0000 C CNN
+F 1 "2x5_2.54mm" H 6150 4676 50  0000 C CNN
+F 2 "Connector_PinHeader_2.54mm:PinHeader_2x05_P2.54mm_Vertical" H 6100 4350 50  0001 C CNN
+F 3 "~" H 6100 4350 50  0001 C CNN
+	1    6100 4350
 	1    0    0    -1
 $EndComp

Commit message: RevB update
Parts:
- J_DATA1: footprint Connector_PinHeader_2.54mm:PinHeader_2x05_P2.54mm_Vertical -> Connector_PinHeader_2.54mm:PinHeader_2x05_P2.54mm_Horizontal
Changed lines of the file:
@@
 GND
 Wire Wire Line
-	6900 4550 6400 4550
+	5400 4550 5900 4550
 Wire Wire Line
-	6900 4450 6400 4450
+	5400 4450 5900 4450
 Wire Wire Line
-	6900 4350 6400 4350
+	5400 4350 5900 4350
 Wire Wire Line
-	6900 4250 6400 4250
+	5400 4250 5900 4250
 Wire Wire Line
-	6900 4150 6400 4150
+	5400 4150 5900 4150
 Wire Wire Line
-	5900 4150 5400 4150
+	6400 4150 6900 4150
+Text Label 6900 4150 2    50   ~ 0
+PSON
 Text Label 5400 4150 0    50   ~ 0
-PSON
-Text Label 6900 4150 2    50   ~ 0
 ISHARE
-Text Label 6900 4250 2    50   ~ 0
+Text Label 5400 4250 0    50   ~ 0
 PSOK
-Text Label 6900 4350 2    50   ~ 0
+Text Label 5400 4350 0    50   ~ 0
 PRESENT
-Text Label 6900 4450 2    50   ~ 0
+Text Label 5400 4450 0    50   ~ 0
 12VSB
-Text Label 6900 4550 2    50   ~ 0
+Text Label 5400 4550 0    50   ~ 0
 PSINTERRUPT
 Wire Wire Line
-	5900 4450 5400 4450
+	6400 4450 6900 4450
 Wire Wire Line
-	5900 4350 5400 4350
+	6400 4350 6900 4350
 Wire Wire Line
-	5900 4250 5400 4250
-Text Label 5400 4450 0    50   ~ 0
+	6400 4250 6900 4250
+Text Label 6900 4450 2    50   ~ 0
 ADDR
 Wire Wire Line
-	5900 4550 5200 4550
+	6400 4550 7100 4550
 Wire Wire Line
-	5200 4850 5200 4550
-Text Label 5200 4850 1    50   ~ 0
+	7100 4850 7100 4550
+Text Label 7100 4850 1    50   ~ 0
 GND
-Text Label 5400 4250 0    50   ~ 0
+Text Label 6900 4250 2    50   ~ 0
 SDA
-Text Label 5400 4350 0    50   ~ 0
+Text Label 6900 4350 2    50   ~ 0
 SCL
 $Comp
@@
 F 0 "J_DATA1" H 6150 4767 50  0000 C CNN
 F 1 "2x5_2.54mm" H 6150 4676 50  0000 C CNN
-F 2 "Connector_PinHeader_2.54mm:PinHeader_2x05_P2.54mm_Vertical" H 6100 4350 50  0001 C CNN
+F 2 "Connector_PinHeader_2.54mm:PinHeader_2x05_P2.54mm_Horizontal" H 6100 4350 50  0001 C CNN
 F 3 "~" H 6100 4350 50  0001 C CNN
 	1    6100 4350
