File: OutputConnectors.sch (KiCad schematic (older format))
At the start: 2 parts

Commit message: layout draft
Parts:
- removed J_GND1, J_VOUT1: 1x6_5.08mm, Samtec HPM-06-02-T-S-RA_1x6:Samtec HPM-06-02-T-S-RA_2x6, symbol Connector_Generic:Conn_01x06
- added J3, J4: Conn_01x01, MountingHole:MountingHole_6.4mm_M6, symbol Connector_Generic:Conn_01x01
Connections:
- wire segments 25 -> 3
Changed lines of the file:
@@
 $EndDescr
 Wire Wire Line
-	5825 2675 5525 2675
+	4600 3000 4300 3000
 Wire Wire Line
-	5425 3575 5425 3775
+	4200 3850 4200 4050
+Wire Wire Line
+	4200 3850 4600 3850
 $Comp
-L Connector_Generic:Conn_01x06 J_VOUT1
-U 1 1 5F02E914
-P 6325 2675
-F 0 "J_VOUT1" H 6404 2667 50  0000 L CNN
-F 1 "1x6_5.08mm" H 6404 2576 50  0000 L CNN
-F 2 "Samtec HPM-06-02-T-S-RA_1x6:Samtec HPM-06-02-T-S-RA_2x6" H 6325 2675 50  0001 C CNN
-F 3 "~" H 6325 2675 50  0001 C CNN
-	1    6325 2675
+L power:GNDS #PWR?
+U 1 1 5F02E93F
+P 4200 4050
+AR Path="/5EFF0F4B/5F02E93F" Ref="#PWR?"  Part="1"
+AR Path="/5F02DF75/5F02E93F" Ref="#PWR04"  Part="1"
+F 0 "#PWR04" H 4200 3800 50  0001 C CNN
+F 1 "GNDS" H 4205 3877 50  0000 C CNN
+F 2 "" H 4200 4050 50  0001 C CNN
+F 3 "" H 4200 4050 50  0001 C CNN
+	1    4200 4050
+	1    0    0    -1
+$EndComp
+Text HLabel 4300 3000 0    50   Input ~ 0
+PSU_VBUS
+$Comp
+L Connector_Generic:Conn_01x01 J3
+U 1 1 5EFFCB36
+P 4800 3000
+F 0 "J3" H 4880 3042 50  0000 L CNN
+F 1 "Conn_01x01" H 4880 2951 50  0000 L CNN
+F 2 "MountingHole:MountingHole_6.4mm_M6" H 4800 3000 50  0001 C CNN
+F 3 "https://docs.rs-online.com/41b5/A700000006757323.pdf" H 4800 3000 50  0001 C CNN
+	1    4800 3000
 	1    0    0    -1
 $EndComp
 $Comp
-L Connector_Generic:Conn_01x06 J_GND1
-U 1 1 5F02E91A
-P 6325 3575
-F 0 "J_GND1" H 6404 3567 50  0000 L CNN
-F 1 "1x6_5.08mm" H 6404 3476 50  0000 L CNN
-F 2 "Samtec HPM-06-02-T-S-RA_1x6:Samtec HPM-06-02-T-S-RA_2x6" H 6325 3575 50  0001 C CNN
-F 3 "~" H 6325 3575 50  0001 C CNN
-	1    6325 3575
+L Connector_Generic:Conn_01x01 J4
+U 1 1 5EFFE270
+P 4800 3850
+F 0 "J4" H 4880 3892 50  0000 L CNN
+F 1 "Conn_01x01" H 4880 3801 50  0000 L CNN
+F 2 "MountingHole:MountingHole_6.4mm_M6" H 4800 3850 50  0001 C CNN
+F 3 "https://docs.rs-online.com/41b5/A700000006757323.pdf" H 4800 3850 50  0001 C CNN
+	1    4800 3850
 	1    0    0    -1
 $EndComp
-Wire Wire Line
-	6125 2475 5825 2475
-Wire Wire Line
-	5825 2475 5825 2575
-Wire Wire Line
-	5825 2975 6125 2975
-Connection ~ 5825 2675
-Wire Wire Line
-	5825 2675 5825 2775
-Wire Wire Line
-	6125 2875 5825 2875
-Connection ~ 5825 2875
-Wire Wire Line
-	5825 2875 5825 2975
-Wire Wire Line
-	6125 2775 5825 2775
-Connection ~ 5825 2775
-Wire Wire Line
-	5825 2775 5825 2875
-Wire Wire Line
-	6125 2675 5825 2675
-Wire Wire Line
-	6125 2575 5825 2575
-Connection ~ 5825 2575
-Wire Wire Line
-	5825 2575 5825 2675
-Wire Wire Line
-	6125 3375 5825 3375
-Wire Wire Line
-	5825 3375 5825 3475
-Wire Wire Line
-	5825 3875 6125 3875
-Connection ~ 5825 3575
-Wire Wire Line
-	5825 3575 5825 3675
-Wire Wire Line
-	6125 3775 5825 3775
-Connection ~ 5825 3775
-Wire Wire Line
-	5825 3775 5825 3875
-Wire Wire Line
-	6125 3675 5825 3675
-Connection ~ 5825 3675
-Wire Wire Line
-	5825 3675 5825 3775
-Wire Wire Line
-	6125 3575 5825 3575
-Wire Wire Line
-	6125 3475 5825 3475
-Connection ~ 5825 3475
-Wire Wire Line
-	5825 3475 5825 3575
-Wire Wire Line
-	5425 3575 5825 3575
-$Comp
-L power:GNDS #PWR?
-U 1 1 5F02E93F
-P 5425 3775
-AR Path="/5EFF0F4B/5F02E93F" Ref="#PWR?"  Part="1"
-AR Path="/5F02DF75/5F02E93F" Ref="#PWR04"  Part="1"
-F 0 "#PWR04" H 5425 3525 50  0001 C CNN
-F 1 "GNDS" H 5430 3602 50  0000 C CNN
-F 2 "" H 5425 3775 50  0001 C CNN
-F 3 "" H 5425 3775 50  0001 C CNN
-	1    5425 3775
-	1    0    0    -1
-$EndComp
-Text HLabel 5525 2675 0    50   Input ~ 0
-PSU_VBUS
 $EndSCHEMATC

Commit message: Completed RevA
Parts:
- J3, J4: footprint MountingHole:MountingHole_6.4mm_M6 -> MountingHole:MountingHole_4.3mm_M4_Pad_Via
Changed lines of the file:
@@
 F 0 "J3" H 4880 3042 50  0000 L CNN
 F 1 "Conn_01x01" H 4880 2951 50  0000 L CNN
-F 2 "MountingHole:MountingHole_6.4mm_M6" H 4800 3000 50  0001 C CNN
+F 2 "MountingHole:MountingHole_4.3mm_M4_Pad_Via" H 4800 3000 50  0001 C CNN
 F 3 "https://docs.rs-online.com/41b5/A700000006757323.pdf" H 4800 3000 50  0001 C CNN
 	1    4800 3000
@@
 F 0 "J4" H 4880 3892 50  0000 L CNN
 F 1 "Conn_01x01" H 4880 3801 50  0000 L CNN
-F 2 "MountingHole:MountingHole_6.4mm_M6" H 4800 3850 50  0001 C CNN
+F 2 "MountingHole:MountingHole_4.3mm_M4_Pad_Via" H 4800 3850 50  0001 C CNN
 F 3 "https://docs.rs-online.com/41b5/A700000006757323.pdf" H 4800 3850 50  0001 C CNN
 	1    4800 3850
