File: HighVoltageControl.sch (KiCad schematic (older format))
At the start: 3 parts, among them Q1 DMG2302U-7, SW1 SW_SPST, U1 NCS1S1203SC

Commit message: UPDATED SWITCH WIRING
Parts:
- removed Q1: DMG2302U-7, Package_TO_SOT_SMD:SOT-23, symbol Device:Q_NMOS_GSD
- added R3: 22K, symbol Device:R
Connections:
- net labels added: PSU_ON, PSU_PRES
- net labels removed: PSU_VBUS, PSU_VDD_SW, PSU_VSS_SW
- wire segments 10 -> 15
Other:
- note added: "1. To “enable” the Main 12Vdc output \nthe PRESENT signal requires to be pulled “high”\nwith respect GND."
- note added: "12VSB PIN CAN PROVIDE 2.5A WHILE PSU IS DISABLED"
- note added: "2. The PS_ON signal can be permanently \nconnected to GND to “enable” the Main 12Vdc output"
- note added: "PSU ENABLE REQUIRES TWO CONDITIONS:\n1. PULLUP PRESENT PIN: TELL PSU IT IS INSERTED INTO ACTIVE SERVER\n2. GND ENABLE PIN"
- moved on the sheet: U1
Changed lines of the file:
@@
 Comment4 ""
 $EndDescr
-Wire Wire Line
-	6000 4500 6000 4050
-Text HLabel 6000 4050 1    50   Input ~ 0
-PSU_VDD_SW
-Wire Wire Line
-	6000 4900 6000 5425
-Text HLabel 6000 5425 3    50   Input ~ 0
-PSU_VSS_SW
-Text HLabel 3325 4700 0    50   Input ~ 0
-PSU_12VSB
-Text HLabel 5875 1650 2    50   Input ~ 0
+Text HLabel 2875 5300 0    50   Input ~ 0
+PSU_ON
+Text HLabel 2975 4575 0    50   Input ~ 0
+PSU_PRES
+Text HLabel 7875 1300 2    50   Input ~ 0
 MCU_3V3
-$Comp
-L Device:Q_NMOS_GSD Q1
-U 1 1 5F03B47D
-P 5900 4700
-F 0 "Q1" H 6105 4791 50  0000 L CNN
-F 1 "DMG2302U-7" H 6105 4700 50  0000 L CNN
-F 2 "Package_TO_SOT_SMD:SOT-23" H 6105 4609 50  0000 L CNN
-F 3 "https://www.mouser.co.uk/datasheet/2/115/DMG2302U-1512446.pdf" H 5900 4700 50  0001 C CNN
-	1    5900 4700
-	1    0    0    -1
-$EndComp
 $Comp
 L Switch:SW_SPST SW1
 U 1 1 5F065BCA
-P 4225 4700
-F 0 "SW1" H 4225 4935 50  0000 C CNN
-F 1 "SW_SPST" H 4225 4844 50  0000 C CNN
-F 2 "" H 4225 4700 50  0001 C CNN
-F 3 "~" H 4225 4700 50  0001 C CNN
-	1    4225 4700
+P 4600 5300
+F 0 "SW1" H 4600 5535 50  0000 C CNN
+F 1 "SW_SPST" H 4600 5444 50  0000 C CNN
+F 2 "" H 4600 5300 50  0001 C CNN
+F 3 "~" H 4600 5300 50  0001 C CNN
+	1    4600 5300
 	1    0    0    -1
 $EndComp
 Wire Wire Line
-	3325 4700 4025 4700
+	2875 5300 4400 5300
 Wire Wire Line
-	4425 4700 5700 4700
+	4800 5300 7350 5300
 $Comp
 L Converter_DCDC:NCS1S1203SC U1
 U 1 1 5F0C9092
-P 4550 1850
-F 0 "U1" H 4550 2317 50  0000 C CNN
-F 1 "NCS1S1203SC" H 4550 2226 50  0000 C CNN
-F 2 "Converter_DCDC:Converter_DCDC_Murata_NCS1SxxxxSC_THT" H 4550 1450 50  0001 C CNN
-F 3 "https://power.murata.com/data/power/ncl/kdc_ncs1.pdf" H 4525 1850 50  0001 C CNN
-	1    4550 1850
+P 6550 1500
+F 0 "U1" H 6550 1967 50  0000 C CNN
+F 1 "NCS1S1203SC" H 6550 1876 50  0000 C CNN
+F 2 "Converter_DCDC:Converter_DCDC_Murata_NCS1SxxxxSC_THT" H 6550 1100 50  0001 C CNN
+F 3 "https://power.murata.com/data/power/ncl/kdc_ncs1.pdf" H 6525 1500 50  0001 C CNN
+	1    6550 1500
 	1    0    0    -1
 $EndComp
 Wire Wire Line
-	4050 1650 2725 1650
-Text HLabel 2725 1650 0    50   Input ~ 0
-PSU_VBUS
-NoConn ~ 4050 1850
+	6050 1300 2825 1300
+NoConn ~ 6050 1500
 Wire Wire Line
-	4050 2050 3725 2050
+	6050 1700 5725 1700
 Wire Wire Line
-	3725 2050 3725 2475
+	5725 1700 5725 2125
 $Comp
 L power:GNDS #PWR05
 U 1 1 5F0CC121
-P 3725 2475
-F 0 "#PWR05" H 3725 2225 50  0001 C CNN
-F 1 "GNDS" H 3730 2302 50  0000 C CNN
-F 2 "" H 3725 2475 50  0001 C CNN
-F 3 "" H 3725 2475 50  0001 C CNN
-	1    3725 2475
+P 5725 2125
+F 0 "#PWR05" H 5725 1875 50  0001 C CNN
+F 1 "GNDS" H 5730 1952 50  0000 C CNN
+F 2 "" H 5725 2125 50  0001 C CNN
+F 3 "" H 5725 2125 50  0001 C CNN
+	1    5725 2125
 	1    0    0    -1
 $EndComp
 Wire Wire Line
-	5050 2050 5550 2050
+	7050 1700 7550 1700
 Wire Wire Line
-	5550 2050 5550 2525
-Text HLabel 5550 2525 3    50   Input ~ 0
+	7550 1700 7550 2175
+Text HLabel 7550 2175 3    50   Input ~ 0
 MCU_GND
 Wire Wire Line
-	5050 1650 5875 1650
+	7050 1300 7875 1300
+$Comp
+L Device:R R3
+U 1 1 5EFD85AF
+P 7350 4225
+F 0 "R3" V 7250 4225 50  0000 C CNN
+F 1 "22K" V 7350 4225 50  0000 C CNN
+F 2 "" V 7280 4225 50  0001 C CNN
+F 3 "~" H 7350 4225 50  0001 C CNN
+	1    7350 4225
+	-1   0    0    1
+$EndComp
+Wire Wire Line
+	7350 4075 7350 3800
+Text HLabel 7350 3800 1    50   Input ~ 0
+PSU_12VSB
+Wire Wire Line
+	7350 4375 7350 4575
+Wire Wire Line
+	2975 4575 7350 4575
+Text Notes 2525 4925 0    50   ~ 0
+1. To “enable” the Main 12Vdc output \nthe PRESENT signal requires to be pulled “high”\nwith respect GND.
+Wire Wire Line
+	7350 5300 7350 5725
+$Comp
+L power:GNDS #PWR0101
+U 1 1 5EFE358D
+P 7350 5725
+F 0 "#PWR0101" H 7350 5475 50  0001 C CNN
+F 1 "GNDS" H 7355 5552 50  0000 C CNN
+F 2 "" H 7350 5725 50  0001 C CNN
+F 3 "" H 7350 5725 50  0001 C CNN
+	1    7350 5725
+	1    0    0    -1
+$EndComp
+Text Notes 2525 5625 0    50   ~ 0
+2. The PS_ON signal can be permanently \nconnected to GND to “enable” the Main 12Vdc output
+Text HLabel 2725 1300 0    50   Input ~ 0
+PSU_12VSB
+Text Notes 2525 4275 0    50   ~ 0
+PSU ENABLE REQUIRES TWO CONDITIONS:\n1. PULLUP PRESENT PIN: TELL PSU IT IS INSERTED INTO ACTIVE SERVER\n2. GND ENABLE PIN
+Text Notes 2225 1175 0    50   ~ 0
+12VSB PIN CAN PROVIDE 2.5A WHILE PSU IS DISABLED
+$Comp
+L power:PWR_FLAG #FLG?
+U 1 1 5EFFE480
+P 2750 1400
+AR Path="/5EFF0F4B/5EFFE480" Ref="#FLG?"  Part="1"
+AR Path="/5F02F4C5/5EFFE480" Ref="#FLG0103"  Part="1"
+F 0 "#FLG0103" H 2750 1475 50  0001 C CNN
+F 1 "PWR_FLAG" V 2750 1528 50  0000 L CNN
+F 2 "" H 2750 1400 50  0001 C CNN
+F 3 "~" H 2750 1400 50  0001 C CNN
+	1    2750 1400
+	0    -1   -1   0
+$EndComp
+Wire Wire Line
+	2750 1400 2825 1400
+Wire Wire Line
+	2825 1400 2825 1300
+Connection ~ 2825 1300
+Wire Wire Line
+	2825 1300 2725 1300
 $EndSCHEMATC

Commit message: layout draft
Parts:
- removed SW1: SW_SPST, symbol Switch:SW_SPST
- added Q1: DMG2302U, Package_TO_SOT_SMD:SOT-23, symbol Transistor_FET:DMG2302U
- R3: footprint (none) -> Resistor_SMD:R_0805_2012Metric_Pad1.15x1.40mm_HandSolder
Connections:
- net labels added: MCU_SW
- wire segments 15 -> 16
Other:
- moved on the sheet: R3, U1
Changed lines of the file:
@@
 Comment4 ""
 $EndDescr
-Text HLabel 2875 5300 0    50   Input ~ 0
+Text HLabel 2125 3850 0    50   Input ~ 0
 PSU_ON
-Text HLabel 2975 4575 0    50   Input ~ 0
+Text HLabel 2225 2000 0    50   Input ~ 0
 PSU_PRES
-Text HLabel 7875 1300 2    50   Input ~ 0
+Text HLabel 5825 5950 2    50   Input ~ 0
 MCU_3V3
+Wire Wire Line
+	2125 3850 3650 3850
+Wire Wire Line
+	4050 3850 6600 3850
 $Comp
-L Switch:SW_SPST SW1
-U 1 1 5F065BCA
-P 4600 5300
-F 0 "SW1" H 4600 5535 50  0000 C CNN
-F 1 "SW_SPST" H 4600 5444 50  0000 C CNN
-F 2 "" H 4600 5300 50  0001 C CNN
-F 3 "~" H 4600 5300 50  0001 C CNN
-	1    4600 5300
+L Converter_DCDC:NCS1S1203SC U1
+U 1 1 5F0C9092
+P 4500 6150
+F 0 "U1" H 4500 6617 50  0000 C CNN
+F 1 "NCS1S1203SC" H 4500 6526 50  0000 C CNN
+F 2 "Converter_DCDC:Converter_DCDC_Murata_NCS1SxxxxSC_THT" H 4500 5750 50  0001 C CNN
+F 3 "https://power.murata.com/data/power/ncl/kdc_ncs1.pdf" H 4475 6150 50  0001 C CNN
+	1    4500 6150
 	1    0    0    -1
 $EndComp
 Wire Wire Line
-	2875 5300 4400 5300
+	4000 5950 2425 5950
+NoConn ~ 4000 6150
 Wire Wire Line
-	4800 5300 7350 5300
+	4000 6350 3650 6350
+Wire Wire Line
+	3650 6350 3650 6775
 $Comp
-L Converter_DCDC:NCS1S1203SC U1
-U 1 1 5F0C9092
-P 6550 1500
-F 0 "U1" H 6550 1967 50  0000 C CNN
-F 1 "NCS1S1203SC" H 6550 1876 50  0000 C CNN
-F 2 "Converter_DCDC:Converter_DCDC_Murata_NCS1SxxxxSC_THT" H 6550 1100 50  0001 C CNN
-F 3 "https://power.murata.com/data/power/ncl/kdc_ncs1.pdf" H 6525 1500 50  0001 C CNN
-	1    6550 1500
+L power:GNDS #PWR05
+U 1 1 5F0CC121
+P 3650 6775
+F 0 "#PWR05" H 3650 6525 50  0001 C CNN
+F 1 "GNDS" H 3655 6602 50  0000 C CNN
+F 2 "" H 3650 6775 50  0001 C CNN
+F 3 "" H 3650 6775 50  0001 C CNN
+	1    3650 6775
 	1    0    0    -1
 $EndComp
 Wire Wire Line
-	6050 1300 2825 1300
-NoConn ~ 6050 1500
+	5000 6350 5500 6350
 Wire Wire Line
-	6050 1700 5725 1700
-Wire Wire Line
-	5725 1700 5725 2125
-$Comp
-L power:GNDS #PWR05
-U 1 1 5F0CC121
-P 5725 2125
-F 0 "#PWR05" H 5725 1875 50  0001 C CNN
-F 1 "GNDS" H 5730 1952 50  0000 C CNN
-F 2 "" H 5725 2125 50  0001 C CNN
-F 3 "" H 5725 2125 50  0001 C CNN
-	1    5725 2125
-	1    0    0    -1
-$EndComp
-Wire Wire Line
-	7050 1700 7550 1700
-Wire Wire Line
-	7550 1700 7550 2175
-Text HLabel 7550 2175 3    50   Input ~ 0
+	5500 6350 5500 6825
+Text HLabel 5500 6825 3    50   Input ~ 0
 MCU_GND
 Wire Wire Line
-	7050 1300 7875 1300
+	5000 5950 5825 5950
 $Comp
 L Device:R R3
 U 1 1 5EFD85AF
-P 7350 4225
-F 0 "R3" V 7250 4225 50  0000 C CNN
-F 1 "22K" V 7350 4225 50  0000 C CNN
-F 2 "" V 7280 4225 50  0001 C CNN
-F 3 "~" H 7350 4225 50  0001 C CNN
-	1    7350 4225
+P 6600 1675
+F 0 "R3" V 6500 1675 50  0000 C CNN
+F 1 "22K" V 6600 1675 50  0000 C CNN
+F 2 "Resistor_SMD:R_0805_2012Metric_Pad1.15x1.40mm_HandSolder" V 6530 1675 50  0001 C CNN
+F 3 "~" H 6600 1675 50  0001 C CNN
+	1    6600 1675
 	-1   0    0    1
 $EndComp
 Wire Wire Line
-	7350 4075 7350 3800
-Text HLabel 7350 3800 1    50   Input ~ 0
+	6600 1525 6600 1250
+Text HLabel 6600 1250 1    50   Input ~ 0
 PSU_12VSB
 Wire Wire Line
-	7350 4375 7350 4575
+	6600 1825 6600 2000
 Wire Wire Line
-	2975 4575 7350 4575
-Text Notes 2525 4925 0    50   ~ 0
+	2225 2000 6600 2000
+Text Notes 1775 2375 0    50   ~ 0
 1. To “enable” the Main 12Vdc output \nthe PRESENT signal requires to be pulled “high”\nwith respect GND.
 Wire Wire Line
-	7350 5300 7350 5725
+	6600 3850 6600 4275
 $Comp
 L power:GNDS #PWR0101
 U 1 1 5EFE358D
-P 7350 5725
-F 0 "#PWR0101" H 7350 5475 50  0001 C CNN
-F 1 "GNDS" H 7355 5552 50  0000 C CNN
-F 2 "" H 7350 5725 50  0001 C CNN
-F 3 "" H 7350 5725 50  0001 C CNN
-	1    7350 5725
+P 6600 4275
+F 0 "#PWR0101" H 6600 4025 50  0001 C CNN
+F 1 "GNDS" H 6605 4102 50  0000 C CNN
+F 2 "" H 6600 4275 50  0001 C CNN
+F 3 "" H 6600 4275 50  0001 C CNN
+	1    6600 4275
 	1    0    0    -1
 $EndComp
-Text Notes 2525 5625 0    50   ~ 0
+Text Notes 1775 4175 0    50   ~ 0
 2. The PS_ON signal can be permanently \nconnected to GND to “enable” the Main 12Vdc output
-Text HLabel 2725 1300 0    50   Input ~ 0
+Text HLabel 2325 5950 0    50   Input ~ 0
 PSU_12VSB
-Text Notes 2525 4275 0    50   ~ 0
+Text Notes 1775 1725 0    50   ~ 0
 PSU ENABLE REQUIRES TWO CONDITIONS:\n1. PULLUP PRESENT PIN: TELL PSU IT IS INSERTED INTO ACTIVE SERVER\n2. GND ENABLE PIN
-Text Notes 2225 1175 0    50   ~ 0
+Text Notes 1825 5825 0    50   ~ 0
 12VSB PIN CAN PROVIDE 2.5A WHILE PSU IS DISABLED
 $Comp
 L power:PWR_FLAG #FLG?
 U 1 1 5EFFE480
-P 2750 1400
+P 2350 6050
 AR Path="/5EFF0F4B/5EFFE480" Ref="#FLG?"  Part="1"
 AR Path="/5F02F4C5/5EFFE480" Ref="#FLG0103"  Part="1"
-F 0 "#FLG0103" H 2750 1475 50  0001 C CNN
-F 1 "PWR_FLAG" V 2750 1528 50  0000 L CNN
-F 2 "" H 2750 1400 50  0001 C CNN
-F 3 "~" H 2750 1400 50  0001 C CNN
-	1    2750 1400
+F 0 "#FLG0103" H 2350 6125 50  0001 C CNN
+F 1 "PWR_FLAG" V 2350 6178 50  0000 L CNN
+F 2 "" H 2350 6050 50  0001 C CNN
+F 3 "~" H 2350 6050 50  0001 C CNN
+	1    2350 6050
 	0    -1   -1   0
 $EndComp
 Wire Wire Line
-	2750 1400 2825 1400
+	2350 6050 2425 6050
 Wire Wire Line
-	2825 1400 2825 1300
-Connection ~ 2825 1300
+	2425 6050 2425 5950
+Connection ~ 2425 5950
 Wire Wire Line
-	2825 1300 2725 1300
+	2425 5950 2325 5950
+$Comp
+L Transistor_FET:DMG2302U Q1
+U 1 1 5F001BDB
+P 3850 3750
+F 0 "Q1" V 3600 3250 50  0000 C CNN
+F 1 "DMG2302U" V 3700 3250 50  0000 C CNN
+F 2 "Package_TO_SOT_SMD:SOT-23" H 4050 3675 50  0001 L CIN
+F 3 "http://www.diodes.com/assets/Datasheets/DMG2302U.pdf" H 3850 3750 50  0001 L CNN
+	1    3850 3750
+	0    1    1    0
+$EndComp
+Wire Wire Line
+	3850 3550 3850 3400
+Text HLabel 3850 3400 1    50   Input ~ 0
+MCU_SW
 $EndSCHEMATC
