File: RevB/MCU.sch (KiCad schematic (older format))
At the start: 18 parts, among them J1 Conn_01x05, J2 Conn_01x14, U2 STM32F072RBTx

Commit message: hw update
updated revb. Added board connectors for device stacking
Parts:
- J1: footprint Connector_PinHeader_2.54mm:PinHeader_1x05_P2.54mm_Horizontal -> Connector_PinHeader_2.54mm:PinHeader_1x05_P2.54mm_Vertical
Changed lines of the file:
@@
 F 0 "J1" H 2043 10542 50  0000 C CNN
 F 1 "Conn_01x05" H 2043 10451 50  0000 C CNN
-F 2 "Connector_PinHeader_2.54mm:PinHeader_1x05_P2.54mm_Horizontal" H 2125 10125 50  0001 C CNN
+F 2 "Connector_PinHeader_2.54mm:PinHeader_1x05_P2.54mm_Vertical" H 2125 10125 50  0001 C CNN
 F 3 "~" H 2125 10125 50  0001 C CNN
 	1    2125 10125
